File: Arduino Shield/Shield.sch (EAGLE design)
At the start: 18 parts, among them IC1 317T, IC2 317T

Commit message: Разводка платы
Parts:
- removed 750: 910, resistor:R-EU_R0805
- removed IOH: 10x1F-H8.5, pinhead:PINHD-1X8
- removed POWER: 8x1F-H8.5, pinhead:PINHD-1X6
- removed X1: (no value), SD card breakout:SDCARDEXTDEVICE
- added AD1: ANALOG_SH, SmartPrj:PINHD-1X6
- added C1, C3: 0.1u, resistor:C-EUC0805
- added C2, C4, C5: 1u/50V, resistor:CPOL-EUE3.5-8
- added IOH1: POWER_AR, pinhead:PINHD-1X8
- added IOH2: POWER_SH, pinhead:PINHD-1X8
- added IOL1: PIN2_SH, SmartPrj:PINHD-1X8
- added JP1: PIN_AR, pinhead:PINHD-1X10
- added JP2: PIN_SH, pinhead:PINHD-1X10
- added LIGHT, SERVO1, SERVO2, SOUND, V_EXT_IN, WINCH: (no value), pinhead:PINHD-1X2
- added U$1: (no value), SD_card:SDCARDVAR2
- added V_IN_JMP: (no value), pinhead:PINHD-1X3
- AD: value 6x1F-H8.5 -> ANALOG_AR
- IOL: value 8x1F-H8.5 -> PIN2_AR
- R10: value 240 -> 1.1k
Connections:
- removed net V_INPUT: POWER.6
- new net 10~: JP1.8, JP2.8
- new net 3~: IOL.4, IOL1.4
- new net 5~: IOL.6, IOL1.6
- new net 6~: IOL.7, IOL1.7
- new net 7V: C2.+, IC2.VO, R9.1, WINCH.2
- new net 9~: JP1.9, JP2.9
- new net A1: AD.2, AD1.2
- new net A2: AD.3, AD1.3
- new net A3: AD.4, AD1.4
- new net A4: AD.5, AD1.5
- new net A5: AD.6, AD1.6
- new net AO: AD.1, AD1.1
- new net AREF: JP1.3, JP2.3
- new net IOREF: IOH1.7, IOH2.7
- new net PIN2: IOL.3, IOL1.3
- new net PIN7: IOL.8, IOL1.8
- new net PIN8: JP1.10, JP2.10
- new net RX0: IOL.1, IOL1.1
- new net SCL: JP1.1, JP2.1
- new net SDA: JP1.2, JP2.2
- new net TX1: IOL.2, IOL1.2
- new net V_EXT_IN: V_EXT_IN.1, V_IN_JMP.3
- new net V_IN_ARD: IOH1.1, IOH2.1, V_IN_JMP.1
- net 3.3V: now also IOH1.5, IOH2.5, U$1.VCC; no longer POWER.2, X1.VDD(VCC)
- net 5V: now also IOH1.4, IOH2.4; no longer IC2.VO, POWER.3, R9.1
- net 6V: now also C4.+, SERVO1.2, SERVO2.2
- net GND: now also C1.2, C2.-, C3.2, C4.-, C5.-, IOH1.2, IOH1.3, IOH2.2, IOH2.3, JP1.4, JP2.4, LIGHT.1, R10.2, SERVO1.1, SERVO2.1, SOUND.1, U$1.GND, U$1.GND1, V_EXT_IN.2, WINCH.1; no longer 750.2, POWER.4, POWER.5, X1.VSS1(GND), X1.VSS2(GND)
- net N$2: now also R10.1; no longer 750.1
- net PIN11: now also JP1.7, JP2.7; no longer IOH.4
- net PIN12: now also JP1.6, JP2.6, U$1.DO; no longer IOH.5, X1.DATA0(DO)
- net PIN13: now also JP1.5, JP2.5; no longer IOH.6
- net PIN4: now also IOL1.5
- net RESET: now also IOH1.6, IOH2.6; no longer POWER.1
- net SD_CLK: now also U$1.SCK; no longer X1.CLK(CLK)
- net SD_CS: now also U$1.CS; no longer X1.CD/DATA3(CS/CD)
- net SD_DI: now also U$1.DI; no longer X1.CMD(DI)
- net V_IN: now also C1.1, C3.1, C5.+, LIGHT.2, SOUND.2, V_IN_JMP.2
Other:
- note added: "Input_pins"
- note added: "Output_pins"
- note added: "SD_Card_module"
- note added: "V_out"
- note added: "Voltage_regulator"
- moved on the sheet: AD, IOL, R1, R10, R2, R3, R4, R5, R6
